Commit message: Add SLAM Toolbox integration, custom Gazebo room, TF fixes, diff drive controller and mapping support

File: src/simple_mobile_robot/urdf/simple_robot.urdf.xacro (robot description, xacro)
@@ -108,4 +108,36 @@
   <dynamics damping="2.0"/>
  </joint>
+ <link name="lidar_mast">
+  <visual>
+    <geometry>
+      <cylinder radius="0.03" length="0.09"/>
+    </geometry>
+    <material name="gray">
+      <color rgba="0.6 0.6 0.6 1"/>
+    </material>
+  </visual>
+  <collision>
+    <geometry>
+      <cylinder radius="0.008" length="0.09"/>
+    </geometry>
+  </collision>
+  <inertial>
+    <mass value="0.05"/>
+    <origin xyz="0 0 0"/>
+    <inertia
+      ixx="0.00001"
+      ixy="0"
+      ixz="0"
+      iyy="0.00001"
+      iyz="0"
+      izz="0.00001"/>
+  </inertial>
+</link>
+<joint name="lidar_mast_joint" type="fixed">
+  <parent link="base_link"/>
+  <child link="lidar_mast"/>
+  <!-- Mast center -->
+  <origin xyz="0 0 0.095" rpy="0 0 0"/>
+</joint>
  <link name="lidar_link">
   <visual>
@@ -134,9 +166,10 @@
   </collision>
  </link>
- <joint name="lidar_joint" type="fixed">
-  <parent link="base_link"/>
+<joint name="lidar_joint" type="fixed">
+  <parent link="lidar_mast"/>
   <child link="lidar_link"/>
-  <origin xyz="0 0 0.075" rpy="0 0 0"/>
- </joint>
+  <!-- LiDAR sits on top of the mast -->
+  <origin xyz="0 0 0.07" rpy="0 0 0"/>
+</joint>
  <link name="depth_camera_link">
   <visual>
@@ -235,11 +268,11 @@
   </inertial>
  </link>
- <joint name="caster_swivel_joint" type="continuous">
+<joint name="caster_swivel_joint" type="continuous">
     <parent link="base_link"/>
     <child link="caster_swivel"/>
     <origin xyz="-0.15 0 -0.045"/>
     <axis xyz="0 0 1"/>
-    <dynamics damping="2.0"/>
- </joint>
+    <dynamics damping="0.05" friction="0.0"/>
+</joint>
  <link name="caster_wheel">
   <visual>
@@ -346,5 +379,5 @@
 </gazebo>
 <gazebo reference="base_link">
-  <sensor name="imu" type="imu">
+  <sensor name="imu_sensor" type="imu">
     <always_on>true</always_on>
     <update_rate>100</update_rate>
@@ -353,4 +386,6 @@
     <enable_metrics>true</enable_metrics>
   </sensor>
+  <kp>1000000</kp>
+  <kd>100</kd>
 </gazebo>
 <gazebo reference="depth_camera_link">
@@ -376,24 +411,20 @@
 </gazebo>
 <gazebo reference="left_wheel">
-  <mu1>1</mu1>
-  <mu2>1</mu2>
-  <kp>1000000</kp>
-  <kd>100</kd>
+  <mu1>10.0</mu1>
+  <mu2>10.0</mu2>
+  <kp>100000</kp>
+  <kd>10</kd>
   <fdir1>0 1 0</fdir1>
 </gazebo>
 <gazebo reference="right_wheel">
-  <mu1>1</mu1>
-  <mu2>1</mu2>
-  <kp>1000000</kp>
-  <kd>100</kd>
+  <mu1>10.0</mu1>
+  <mu2>10.0</mu2>
+  <kp>100000</kp>
+  <kd>10</kd>
   <fdir1>0 1 0</fdir1>
 </gazebo>
-<gazebo reference="base_link">
-    <kp>1000000</kp>
-    <kd>100</kd>
-</gazebo>
 <gazebo reference="caster_wheel">
-    <mu1>0.2</mu1>
-    <mu2>0.2</mu2>
+    <mu1>0.01</mu1>
+    <mu2>0.01</mu2>
     <kp>100000</kp>
     <kd>10</kd>
